Commit message: corrected xacro files

File: manipulator_h_description/urdf/manipulator_h.xacro (robot description, xacro)
@@ -1,11 +1,12 @@
 <?xml version="1.0"?>
 <robot name="robotis_manipulator_h" xmlns:xacro="http://www.ros.org/wiki/xacro">
+  <xacro:property name="prefix" value ="manipulator_h"/>
     <!-- some parameters -->
     <!-- <xacro:property name="pi" value="3.141592654" /> -->
     <!-- Import all Gazebo-customization elements, including Gazebo colors -->
-    <xacro:include filename="$(find manipulator_h_description)/urdf/manipulator_h.gazebo" />
+  <xacro:include filename="$(find manipulator_h_description)/urdf/manipulator_h.gazebo" />
     <!-- Import Rviz colors -->
-    <xacro:include filename="$(find manipulator_h_description)/urdf/materials.xacro" />
-  <xacro:macro name="manipulator_h" params="parent *origin">
+  <xacro:include filename="$(find manipulator_h_description)/urdf/materials.xacro" />
+  <xacro:macro name="manipulator_h" params="parent prefix *origin">
     <!-- Used for fixing robot to Gazebo 'link 1' -->
     <!-- <link name="world">
@@ -16,6 +17,6 @@
       <child link="link1"/>
     </joint> -->
-    <joint name="world_fixed" type="fixed">
-      <xacro:insert_block name="origin" />
+    <joint name="${prefix}_world_fixed" type="fixed">
+      <xacro:insert_block name="origin"/>
       <parent link="${parent}" />
       <child link="link1" />

File: manipulator_h_description/urdf/manipulator_h_ros2_control.urdf.xacro (robot description, xacro)
@@ -2,7 +2,9 @@
 <robot name="manipulator_h" xmlns:xacro="http://ros.org/wiki/xacro">
   <xacro:include filename="$(find manipulator_h_description)/urdf/manipulator_h.xacro" />
+  <xacro:include filename="$(find manipulator_h_description)/urdf/manipulator_h.ros2_control.xacro" />
   <link name="world"/>
   <xacro:manipulator_h parent="world">
     <origin xyz="0 0 0" rpy="0 0 0" />
   </xacro:manipulator_h>
+  <xacro:manipulator_h_ros2_control name="manipulator_h_ros2_control" />
 </robot>
