Commit message: [description] corrected baselink reference

File: manipulator_h_description/urdf/manipulator_h.ros2_control.xacro (robot description, xacro)
@@ -7,5 +7,5 @@
         <param name="usb_port">/dev/ttyUSB0</param>
         <param name="baud_rate">1000000</param>
-        <param name="use_dummy">false</param>
+        <param name="use_dummy">true</param>
       </hardware>
       <joint name="joint1">

File: manipulator_h_description/urdf/manipulator_h.xacro (robot description, xacro)
@@ -1,9 +1,8 @@
 <?xml version="1.0"?>
-<!-- Revolute-Revolute Manipulator -->
 <robot name="robotis_manipulator_h" xmlns:xacro="http://www.ros.org/wiki/xacro">
     <!-- some parameters -->
     <!-- <xacro:property name="pi" value="3.141592654" /> -->
     <!-- Import all Gazebo-customization elements, including Gazebo colors -->
-    <!-- <xacro:include filename="$(find manipulator_h_description)/urdf/manipulator_h.gazebo" /> -->
+    <xacro:include filename="$(find manipulator_h_description)/urdf/manipulator_h.gazebo" />
     <!-- Import Rviz colors -->
     <xacro:include filename="$(find manipulator_h_description)/urdf/materials.xacro" />
@@ -17,5 +16,5 @@
       <child link="link1"/>
     </joint> -->
-    <joint name="origin_to_link1" type="fixed">
+    <joint name="world_fixed" type="fixed">
       <xacro:insert_block name="origin" />
       <parent link="${parent}" />
@@ -28,11 +27,11 @@
         <origin xyz="0 0 0" rpy="0 0 0"/>
         <geometry>
-          <mesh filename="package://manipulator_h_description/meshes/link_1.stl" scale="0.001 0.001 0.001"/>
-        </geometry>
-      </collision>
-      <visual>
-        <origin xyz="0 0 0" rpy="0 0 0"/>
-        <geometry>
-          <mesh filename="package://manipulator_h_description/meshes/link_1.stl" scale="0.001 0.001 0.001"/>
+          <mesh filename="file://$(find manipulator_h_description)/meshes/link_1.stl" scale="0.001 0.001 0.001"/>
+        </geometry>
+      </collision>
+      <visual>
+        <origin xyz="0 0 0" rpy="0 0 0"/>
+        <geometry>
+          <mesh filename="file://$(find manipulator_h_description)/meshes/link_1.stl" scale="0.001 0.001 0.001"/>
         </geometry>
         <material name="white"/>
@@ -70,11 +69,11 @@
         <origin xyz="0 0 0" rpy="0 0 0"/>
         <geometry>
-          <mesh filename="package://manipulator_h_description/meshes/link_2.stl" scale="0.001 0.001 0.001"/>
-        </geometry>
-      </collision>
-      <visual>
-        <origin xyz="0 0 0" rpy="0 0 0"/>
-        <geometry>
-          <mesh filename="package://manipulator_h_description/meshes/link_2.stl" scale="0.001 0.001 0.001"/>
+          <mesh filename="file://$(find manipulator_h_description)/meshes/link_2.stl" scale="0.001 0.001 0.001"/>
+        </geometry>
+      </collision>
+      <visual>
+        <origin xyz="0 0 0" rpy="0 0 0"/>
+        <geometry>
+          <mesh filename="file://$(find manipulator_h_description)/meshes/link_2.stl" scale="0.001 0.001 0.001"/>
         </geometry>
         <material name="white"/>
@@ -112,11 +111,11 @@
         <origin xyz="0 0 0" rpy="0 0 0"/>
         <geometry>
-          <mesh filename="package://manipulator_h_description/meshes/link_3.stl" scale="0.001 0.001 0.001"/>
-        </geometry>
-      </collision>
-      <visual>
-        <origin xyz="0 0 0" rpy="0 0 0"/>
-        <geometry>
-          <mesh filename="package://manipulator_h_description/meshes/link_3.stl" scale="0.001 0.001 0.001"/>
+          <mesh filename="file://$(find manipulator_h_description)/meshes/link_3.stl" scale="0.001 0.001 0.001"/>
+        </geometry>
+      </collision>
+      <visual>
+        <origin xyz="0 0 0" rpy="0 0 0"/>
+        <geometry>
+          <mesh filename="file://$(find manipulator_h_description)/meshes/link_3.stl" scale="0.001 0.001 0.001"/>
         </geometry>
         <material name="white"/>
@@ -154,11 +153,11 @@
         <origin xyz="0 0 0" rpy="0 0 0"/>
         <geometry>
-          <mesh filename="package://manipulator_h_description/meshes/link_4.stl" scale="0.001 0.001 0.001"/>
-        </geometry>
-      </collision>
-      <visual>
-        <origin xyz="0 0 0" rpy="0 0 0"/>
-        <geometry>
-          <mesh filename="package://manipulator_h_description/meshes/link_4.stl" scale="0.001 0.001 0.001"/>
+          <mesh filename="file://$(find manipulator_h_description)/meshes/link_4.stl" scale="0.001 0.001 0.001"/>
+        </geometry>
+      </collision>
+      <visual>
+        <origin xyz="0 0 0" rpy="0 0 0"/>
+        <geometry>
+          <mesh filename="file://$(find manipulator_h_description)/meshes/link_4.stl" scale="0.001 0.001 0.001"/>
         </geometry>
         <material name="white"/>
@@ -196,11 +195,11 @@
         <origin xyz="0 0 0" rpy="0 0 0"/>
         <geometry>
-          <mesh filename="package://manipulator_h_description/meshes/link_5.stl" scale="0.001 0.001 0.001"/>
-        </geometry>
-      </collision>
-      <visual>
-        <origin xyz="0 0 0" rpy="0 0 0"/>
-        <geometry>
-          <mesh filename="package://manipulator_h_description/meshes/link_5.stl" scale="0.001 0.001 0.001"/>
+          <mesh filename="file://$(find manipulator_h_description)/meshes/link_5.stl" scale="0.001 0.001 0.001"/>
+        </geometry>
+      </collision>
+      <visual>
+        <origin xyz="0 0 0" rpy="0 0 0"/>
+        <geometry>
+          <mesh filename="file://$(find manipulator_h_description)/meshes/link_5.stl" scale="0.001 0.001 0.001"/>
         </geometry>
         <material name="white"/>
@@ -238,11 +237,11 @@
         <origin xyz="0 0 0" rpy="0 0 0"/>
         <geometry>
-          <mesh filename="package://manipulator_h_description/meshes/link_6.stl" scale="0.001 0.001 0.001"/>
-        </geometry>
-      </collision>
-      <visual>
-        <origin xyz="0 0 0" rpy="0 0 0"/>
-        <geometry>
-          <mesh filename="package://manipulator_h_description/meshes/link_6.stl" scale="0.001 0.001 0.001"/>
+          <mesh filename="file://$(find manipulator_h_description)/meshes/link_6.stl" scale="0.001 0.001 0.001"/>
+        </geometry>
+      </collision>
+      <visual>
+        <origin xyz="0 0 0" rpy="0 0 0"/>
+        <geometry>
+          <mesh filename="file://$(find manipulator_h_description)/meshes/link_6.stl" scale="0.001 0.001 0.001"/>
         </geometry>
         <material name="white"/>
@@ -280,11 +279,11 @@
         <origin xyz="0 0 0" rpy="0 0 0"/>
         <geometry>
-          <mesh filename="package://manipulator_h_description/meshes/end_link.stl" scale="0.001 0.001 0.001"/>
-        </geometry>
-      </collision>
-      <visual>
-        <origin xyz="0 0 0" rpy="0 0 0"/>
-        <geometry>
-          <mesh filename="package://manipulator_h_description/meshes/end_link.stl" scale="0.001 0.001 0.001"/>
+          <mesh filename="file://$(find manipulator_h_description)/meshes/end_link.stl" scale="0.001 0.001 0.001"/>
+        </geometry>
+      </collision>
+      <visual>
+        <origin xyz="0 0 0" rpy="0 0 0"/>
+        <geometry>
+          <mesh filename="file://$(find manipulator_h_description)/meshes/end_link.stl" scale="0.001 0.001 0.001"/>
         </geometry>
         <material name="white"/>

Commit message: added param true/false to use dummy motors for "move_group.launch.py"

File: manipulator_h_description/urdf/manipulator_h.ros2_control.xacro (robot description, xacro)
@@ -1,5 +1,5 @@
 <?xml version="1.0"?>
 <robot xmlns:xacro="http://www.ros.org/wiki/xacro">
-  <xacro:macro name="manipulator_h_ros2_control" params="name">
+  <xacro:macro name="manipulator_h_ros2_control" params="name use_dummy:='true'">
     <ros2_control name="${name}" type="system">
       <hardware>
@@ -7,5 +7,5 @@
         <param name="usb_port">/dev/ttyUSB0</param>
         <param name="baud_rate">1000000</param>
-        <param name="use_dummy">true</param>
+        <param name="use_dummy">${use_dummy}</param>
       </hardware>
       <joint name="joint1">

File: manipulator_h_description/urdf/manipulator_h_ros2_control.urdf.xacro (robot description, xacro)
@@ -4,7 +4,7 @@
   <xacro:include filename="$(find manipulator_h_description)/urdf/manipulator_h.ros2_control.xacro" />
   <link name="world"/>
-  <xacro:manipulator_h parent="world">
+  <xacro:manipulator_h parent="world" prefix="arm">
     <origin xyz="0 0 0" rpy="0 0 0" />
   </xacro:manipulator_h>
-  <xacro:manipulator_h_ros2_control name="manipulator_h_ros2_control" />
+  <xacro:manipulator_h_ros2_control name="manipulator_h_ros2_control" use_dummy="true"/>
 </robot>
